Commit message: added xacro for lite6 arm

File: urdf/arm/lite6.urdf (robot description, URDF)
Before this commit: robot my_robot, 8 links, 7 joints
Links:
- link link1: geometry collision mesh filename=file://$(find lynx_quanta)/meshes/arm/link1.stl; visual mesh filename=file://$(find lynx_quanta)/meshes/arm/link1.stl
- link link2: geometry collision mesh filename=file://$(find lynx_quanta)/meshes/arm/link2.stl; visual mesh filename=file://$(find lynx_quanta)/meshes/arm/link2.stl
- link link3: geometry collision mesh filename=file://$(find lynx_quanta)/meshes/arm/link3.stl; visual mesh filename=file://$(find lynx_quanta)/meshes/arm/link3.stl
- link link4: geometry collision mesh filename=file://$(find lynx_quanta)/meshes/arm/link4.stl; visual mesh filename=file://$(find lynx_quanta)/meshes/arm/link4.stl
- link link5: geometry collision mesh filename=file://$(find lynx_quanta)/meshes/arm/link5.stl; visual mesh filename=file://$(find lynx_quanta)/meshes/arm/link5.stl
- link link6: geometry collision mesh filename=file://$(find lynx_quanta)/meshes/arm/link6.stl; visual mesh filename=file://$(find lynx_quanta)/meshes/arm/link6.stl
- link link_base: geometry collision mesh filename=file://$(find lynx_quanta)/meshes/arm/base.stl; visual mesh filename=file://$(find lynx_quanta)/meshes/arm/base.stl
