Commit message: changed limits and damping frictions for arm

File: urdf/m20_with_arm/m20_with_piper.urdf (robot description, URDF)
Before this commit: robot m20_with_piper, 33 links, 32 joints
Joints:
- joint arm_joint2: limit lower=0 upper=3.14 effort=100 velocity=5 -> lower=0 upper=3.4034 effort=100 velocity=3.403
- joint arm_joint4: limit lower=-1.745 upper=1.745 effort=100 velocity=5 -> lower=-1.7453 upper=1.9548 effort=100 velocity=3.927
- joint arm_joint6: limit lower=-2.0944 upper=2.0944 effort=100 velocity=3 -> lower=-2.9671 upper=2.9671 effort=100 velocity=3.927
- joint arm_joint7: limit lower=0 upper=0.035 effort=10 velocity=1 -> lower=0.0 upper=0.035 effort=120 velocity=0.5
- joint arm_joint8: axis 0 0 -1 -> 0 0 1; limit lower=-0.035 upper=0 effort=10 velocity=1 -> lower=0.0 upper=0.035 effort=120 velocity=0.5
